File: ledboard2/ledboard2.sch (KiCad schematic (older format))
At the start: 105 parts, among them P1 CONN_01X03, P2 CONN_01X03, U1 NEOPIXEL, U10 NEOPIXEL, U100 NEOPIXEL, U11 NEOPIXEL, U12 NEOPIXEL, U13 NEOPIXEL, U14 NEOPIXEL, U15 NEOPIXEL, U16 NEOPIXEL, U17 NEOPIXEL, U18 NEOPIXEL, U19 NEOPIXEL, U2 NEOPIXEL, U20 NEOPIXEL, U21 NEOPIXEL, U22 NEOPIXEL, U23 NEOPIXEL, U24 NEOPIXEL, U25 NEOPIXEL, U26 NEOPIXEL, U27 NEOPIXEL, U28 NEOPIXEL, U29 NEOPIXEL, U3 NEOPIXEL, U30 NEOPIXEL, U31 NEOPIXEL, U32 NEOPIXEL, U33 NEOPIXEL, U34 NEOPIXEL, U35 NEOPIXEL, U36 NEOPIXEL, U37 NEOPIXEL, U38 NEOPIXEL, U39 NEOPIXEL, U4 NEOPIXEL, U40 NEOPIXEL, U41 NEOPIXEL, U42 NEOPIXEL, U43 NEOPIXEL, U44 NEOPIXEL, U45 NEOPIXEL, U46 NEOPIXEL, U47 NEOPIXEL, U48 NEOPIXEL, U49 NEOPIXEL, U5 NEOPIXEL, U50 NEOPIXEL, U51 NEOPIXEL, U52 NEOPIXEL, U53 NEOPIXEL, U54 NEOPIXEL, U55 NEOPIXEL, U56 NEOPIXEL, U57 NEOPIXEL, U58 NEOPIXEL, U59 NEOPIXEL, U6 NEOPIXEL, U60 NEOPIXEL, U61 NEOPIXEL, U62 NEOPIXEL, U63 NEOPIXEL, U64 NEOPIXEL, U65 NEOPIXEL, U66 NEOPIXEL, U67 NEOPIXEL, U68 NEOPIXEL, U69 NEOPIXEL, U7 NEOPIXEL, U70 NEOPIXEL, U71 NEOPIXEL, U72 NEOPIXEL, U73 NEOPIXEL, U74 NEOPIXEL, U75 NEOPIXEL, U76 NEOPIXEL, U77 NEOPIXEL, U78 NEOPIXEL, U79 NEOPIXEL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

Commit message: Increase NeoPixel hole sizes and add bigger capacitor.
Parts:
- added C3: CP, symbol CP
Connections:
- net +5V: now also C3.1
- net GND: now also C3.2
Changed lines of the file:
@@
 LIBS:valves
 LIBS:ledboard2
+LIBS:ledboard2-cache
 EELAYER 25 0
 EELAYER END
@@
 Connection ~ 10200 1800
 $Comp
-L +5V #PWR01
+L +5V #PWR3
 U 1 1 559EEA2D
 P 1550 900
-F 0 "#PWR01" H 1550 750 50  0001 C CNN
+F 0 "#PWR3" H 1550 750 50  0001 C CNN
 F 1 "+5V" H 1550 1040 50  0000 C CNN
 F 2 "" H 1550 900 60  0000 C CNN
@@
 Connection ~ 9150 1050
 $Comp
-L GND #PWR02
+L GND #PWR12
 U 1 1 559F132F
 P 10200 6150
-F 0 "#PWR02" H 10200 5900 50  0001 C CNN
+F 0 "#PWR12" H 10200 5900 50  0001 C CNN
 F 1 "GND" H 10200 6000 50  0000 C CNN
 F 2 "" H 10200 6150 60  0000 C CNN
@@
 	5600 6850 5650 6850
 $Comp
-L +5V #PWR03
+L +5V #PWR10
 U 1 1 55A02828
 P 5150 6900
-F 0 "#PWR03" H 5150 6750 50  0001 C CNN
+F 0 "#PWR10" H 5150 6750 50  0001 C CNN
 F 1 "+5V" H 5150 7040 50  0000 C CNN
 F 2 "" H 5150 6900 60  0000 C CNN
@@
 $EndComp
 $Comp
-L GND #PWR04
+L GND #PWR11
 U 1 1 55A02906
 P 5150 7100
-F 0 "#PWR04" H 5150 6850 50  0001 C CNN
+F 0 "#PWR11" H 5150 6850 50  0001 C CNN
 F 1 "GND" H 5150 6950 50  0000 C CNN
 F 2 "" H 5150 7100 60  0000 C CNN
@@
 $EndComp
 $Comp
-L +5V #PWR05
+L +5V #PWR1
 U 1 1 55A06658
 P 1150 6700
-F 0 "#PWR05" H 1150 6550 50  0001 C CNN
+F 0 "#PWR1" H 1150 6550 50  0001 C CNN
 F 1 "+5V" H 1150 6840 50  0000 C CNN
 F 2 "" H 1150 6700 60  0000 C CNN
@@
 $EndComp
 $Comp
-L GND #PWR06
+L GND #PWR2
 U 1 1 55A06738
 P 1150 7200
-F 0 "#PWR06" H 1150 6950 50  0001 C CNN
+F 0 "#PWR2" H 1150 6950 50  0001 C CNN
 F 1 "GND" H 1150 7050 50  0000 C CNN
 F 2 "" H 1150 7200 60  0000 C CNN
@@
 $EndComp
 $Comp
-L +5V #PWR07
+L +5V #PWR4
 U 1 1 55A0783D
 P 1600 6700
-F 0 "#PWR07" H 1600 6550 50  0001 C CNN
+F 0 "#PWR4" H 1600 6550 50  0001 C CNN
 F 1 "+5V" H 1600 6840 50  0000 C CNN
 F 2 "" H 1600 6700 60  0000 C CNN
@@
 $EndComp
 $Comp
-L GND #PWR08
+L GND #PWR5
 U 1 1 55A07843
 P 1600 7200
-F 0 "#PWR08" H 1600 6950 50  0001 C CNN
+F 0 "#PWR5" H 1600 6950 50  0001 C CNN
 F 1 "GND" H 1600 7050 50  0000 C CNN
 F 2 "" H 1600 7200 60  0000 C CNN
@@
 	3800 6850 3850 6850
 $Comp
-L +5V #PWR09
+L +5V #PWR8
 U 1 1 55A09C2E
 P 3350 6900
-F 0 "#PWR09" H 3350 6750 50  0001 C CNN
+F 0 "#PWR8" H 3350 6750 50  0001 C CNN
 F 1 "+5V" H 3350 7040 50  0000 C CNN
 F 2 "" H 3350 6900 60  0000 C CNN
@@
 $EndComp
 $Comp
-L GND #PWR010
+L GND #PWR9
 U 1 1 55A09C34
 P 3350 7100
-F 0 "#PWR010" H 3350 6850 50  0001 C CNN
+F 0 "#PWR9" H 3350 6850 50  0001 C CNN
 F 1 "GND" H 3350 6950 50  0000 C CNN
 F 2 "" H 3350 7100 60  0000 C CNN
@@
 Wire Wire Line
 	1150 1300 1200 1300
+$Comp
+L CP C3
+U 1 1 55EE1E42
+P 2100 6950
+F 0 "C3" H 2125 7050 50  0000 L CNN
+F 1 "CP" H 2125 6850 50  0000 L CNN
+F 2 "" H 2138 6800 30  0000 C CNN
+F 3 "" H 2100 6950 60  0000 C CNN
+	1    2100 6950
+	1    0    0    -1
+$EndComp
+$Comp
+L +5V #PWR6
+U 1 1 55EE2514
+P 2100 6700
+F 0 "#PWR6" H 2100 6550 50  0001 C CNN
+F 1 "+5V" H 2100 6840 50  0000 C CNN
+F 2 "" H 2100 6700 60  0000 C CNN
+F 3 "" H 2100 6700 60  0000 C CNN
+	1    2100 6700
+	1    0    0    -1
+$EndComp
+$Comp
+L GND #PWR7
+U 1 1 55EE25FC
+P 2100 7200
+F 0 "#PWR7" H 2100 6950 50  0001 C CNN
+F 1 "GND" H 2100 7050 50  0000 C CNN
+F 2 "" H 2100 7200 60  0000 C CNN
+F 3 "" H 2100 7200 60  0000 C CNN
+	1    2100 7200
+	1    0    0    -1
+$EndComp
+Wire Wire Line
+	2100 6700 2100 6800
+Wire Wire Line
+	2100 7100 2100 7200
 $EndSCHEMATC
